File: RelayDriverShield8.brd (EAGLE design)
At the start: 62.2 x 69.8 mm, 75 parts, among them IC1 MCP23017SO, J1 Analog, J2 POWER, J3 Digital_0_7, J4 M100.1, J5 ICSPPTH, J7 PWR SELECT, Q1 2N7002, Q2 2N7002, Q3 2N7002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

Commit message: Updated SKU and schematic PDF
Other:
- board text added: "(c) 2012-14 Freetronics Pty Ltd"
- board text removed: "(c) 2012 Freetronics Pty Ltd"
Changed lines of the file:
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@@
 <layer number="22" name="bPlace" color="14" fill="1" visible="yes" active="yes"/>
 <layer number="23" name="tOrigins" color="15" fill="1" visible="yes" active="yes"/>
-<layer number="24" name="bOrigins" color="15" fill="1" visible="no" active="yes"/>
+<layer number="24" name="bOrigins" color="15" fill="1" visible="yes" active="yes"/>
 <layer number="25" name="tNames" color="7" fill="1" visible="yes" active="yes"/>
 <layer number="26" name="bNames" color="7" fill="1" visible="no" active="yes"/>
@@
 <wire x1="18.034" y1="17.653" x2="19.812" y2="16.129" width="0.4064" layer="22" curve="90.012891"/>
 <circle x="40.132" y="22.098" radius="0.254" width="0.4064" layer="21"/>
-<text x="54.864" y="56.642" size="1.4224" layer="22" font="vector" ratio="16" rot="SMR0">(c) 2012 Freetronics Pty Ltd</text>
+<text x="56.896" y="56.642" size="1.4224" layer="22" font="vector" ratio="16" rot="SMR0">(c) 2012-14 Freetronics Pty Ltd</text>
 <text x="25.654" y="4.191" size="0.8128" layer="21" font="vector" ratio="15">RST</text>
 <text x="28.194" y="4.572" size="0.8128" layer="21" font="vector" ratio="15">3V3</text>

Commit message: Added solder jumper to link IOREF and 5V
Parts:
- added SJ4: (no value), freetronics-jon:SJ
Connections:
- net 5V: now also SJ4.2
- net IOREF: now also SJ4.1
Routing:
- net 5V: track 0.00 -> 7.28 mm
Other:
- board text added: "IOREF"
- board text added: "Released under the TAPR Open Hardware License: tapr.org/OHL"
- board text added: "TO 5V"
Changed lines of the file:
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@@
 <layer number="23" name="tOrigins" color="15" fill="1" visible="yes" active="yes"/>
 <layer number="24" name="bOrigins" color="15" fill="1" visible="yes" active="yes"/>
-<layer number="25" name="tNames" color="7" fill="1" visible="yes" active="yes"/>
+<layer number="25" name="tNames" color="7" fill="1" visible="no" active="yes"/>
 <layer number="26" name="bNames" color="7" fill="1" visible="no" active="yes"/>
 <layer number="27" name="tValues" color="7" fill="1" visible="no" active="yes"/>
@@
 <layer number="49" name="Reference" color="7" fill="1" visible="no" active="yes"/>
 <layer number="50" name="dxf" color="7" fill="1" visible="no" active="yes"/>
-<layer number="51" name="tDocu" color="6" fill="1" visible="yes" active="yes"/>
+<layer number="51" name="tDocu" color="6" fill="1" visible="no" active="yes"/>
 <layer number="52" name="bDocu" color="7" fill="1" visible="no" active="yes"/>
 <layer number="53" name="tGND_GNDA" color="7" fill="9" visible="no" active="no"/>
@@
 <wire x1="39.878" y1="28.702" x2="39.37" y2="29.21" width="0.3048" layer="21" curve="90"/>
 <wire x1="39.37" y1="29.21" x2="34.29" y2="29.21" width="0.3048" layer="21"/>
-<text x="54.356" y="29.718" size="1.27" layer="22" font="vector" ratio="15" rot="MR0">0
+<text x="49.022" y="29.718" size="1.27" layer="22" font="vector" ratio="15" rot="MR0">0
 0
 0
@@
 1
 1</text>
-<text x="51.308" y="29.718" size="1.27" layer="22" font="vector" ratio="15" rot="MR0">0
+<text x="45.974" y="29.718" size="1.27" layer="22" font="vector" ratio="15" rot="MR0">0
 0
 1
@@
 1
 1</text>
-<text x="48.26" y="29.718" size="1.27" layer="22" font="vector" ratio="15" rot="MR0">0
+<text x="42.926" y="29.718" size="1.27" layer="22" font="vector" ratio="15" rot="MR0">0
 1
 0
@@
 0
 1</text>
-<text x="45.72" y="29.718" size="1.27" layer="22" font="vector" ratio="15" rot="MR0">0x20
+<text x="54.864" y="29.718" size="1.27" layer="22" font="vector" ratio="15" rot="MR0">0x20
 0x21
 0x22
@@
 0x26
 0x27</text>
-<text x="54.864" y="44.958" size="1.27" layer="22" font="vector" ratio="15" rot="MR0">A2</text>
-<text x="51.816" y="44.958" size="1.27" layer="22" font="vector" ratio="15" rot="MR0">A1</text>
-<text x="48.768" y="44.958" size="1.27" layer="22" font="vector" ratio="15" rot="MR0">A0</text>
-<text x="45.212" y="44.958" size="1.27" layer="22" font="vector" ratio="15" rot="MR0">HEX</text>
+<text x="49.53" y="44.958" size="1.27" layer="22" font="vector" ratio="15" rot="MR0">A2</text>
+<text x="46.482" y="44.958" size="1.27" layer="22" font="vector" ratio="15" rot="MR0">A1</text>
+<text x="43.434" y="44.958" size="1.27" layer="22" font="vector" ratio="15" rot="MR0">A0</text>
+<text x="54.102" y="44.958" size="1.27" layer="22" font="vector" ratio="15" rot="MR0">HEX</text>
 <wire x1="41.402" y1="46.736" x2="40.894" y2="46.228" width="0.254" layer="22" curve="90"/>
 <wire x1="40.894" y1="46.228" x2="40.894" y2="44.704" width="0.254" layer="22"/>
 <wire x1="40.894" y1="44.704" x2="40.894" y2="29.972" width="0.254" layer="22"/>
 <wire x1="40.894" y1="29.972" x2="41.402" y2="29.464" width="0.254" layer="22" curve="90"/>
-<wire x1="41.402" y1="29.464" x2="46.228" y2="29.464" width="0.254" layer="22"/>
-<wire x1="46.228" y1="29.464" x2="54.864" y2="29.464" width="0.254" layer="22"/>
+<wire x1="41.402" y1="29.464" x2="50.038" y2="29.464" width="0.254" layer="22"/>
+<wire x1="50.038" y1="29.464" x2="54.864" y2="29.464" width="0.254" layer="22"/>
 <wire x1="54.864" y1="29.464" x2="55.372" y2="29.972" width="0.254" layer="22" curve="90"/>
 <wire x1="55.372" y1="29.972" x2="55.372" y2="44.704" width="0.254" layer="22"/>
 <wire x1="55.372" y1="44.704" x2="55.372" y2="46.228" width="0.254" layer="22"/>
 <wire x1="55.372" y1="46.228" x2="54.864" y2="46.736" width="0.254" layer="22" curve="90"/>
-<wire x1="54.864" y1="46.736" x2="46.228" y2="46.736" width="0.254" layer="22"/>
-<wire x1="46.228" y1="46.736" x2="41.402" y2="46.736" width="0.254" layer="22"/>
+<wire x1="54.864" y1="46.736" x2="50.038" y2="46.736" width="0.254" layer="22"/>
+<wire x1="50.038" y1="46.736" x2="41.402" y2="46.736" width="0.254" layer="22"/>
 <wire x1="40.894" y1="44.704" x2="55.372" y2="44.704" width="0.254" layer="22"/>
-<wire x1="46.228" y1="46.736" x2="46.228" y2="29.464" width="0.254" layer="22"/>
+<wire x1="50.038" y1="46.736" x2="50.038" y2="29.464" width="0.254" layer="22"/>
 <wire x1="27.686" y1="35.56" x2="27.686" y2="33.274" width="0.3048" layer="22"/>
 <text x="19.05" y="11.43" size="1.27" layer="21" font="vector" ratio="18">A1</text>
@@
 <wire x1="9.144" y1="50.8" x2="9.652" y2="50.292" width="0.3048" layer="21"/>
 <wire x1="9.652" y1="50.292" x2="10.414" y2="51.816" width="0.3048" layer="21"/>
-<text x="19.812" y="28.448" size="1.6764" layer="21" ratio="16">tron.cc/r8</text>
+<text x="17.272" y="32.258" size="1.6764" layer="21" ratio="16" rot="R90">tron.cc/r8</text>
 <rectangle x1="28.956" y1="3.81" x2="29.464" y2="4.318" layer="21"/>
+<text x="56.769" y="53.34" size="1.016" layer="22" font="vector" ratio="17" rot="SMR0">Released under the TAPR Open
+Hardware License: tapr.org/OHL</text>
+<wire x1="29.718" y1="7.366" x2="30.734" y2="7.366" width="0.4064" layer="22"/>
+<wire x1="30.734" y1="7.366" x2="31.75" y2="6.35" width="0.4064" layer="22"/>
+<wire x1="31.75" y1="6.35" x2="31.75" y2="5.334" width="0.4064" layer="22"/>
+<wire x1="26.162" y1="7.366" x2="25.146" y2="7.366" width="0.4064" layer="22"/>
+<wire x1="25.146" y1="7.366" x2="24.13" y2="6.35" width="0.4064" layer="22"/>
+<text x="29.464" y="11.176" size="1.016" layer="22" ratio="15" rot="MR0">LINK</text>
+<text x="29.972" y="9.906" size="1.016" layer="22" ratio="15" rot="MR0">IOREF</text>
+<text x="30.226" y="8.636" size="1.016" layer="22" ratio="15" rot="MR0">TO 5V</text>
 </plain>
 <attributes>
@@
 <attribute name="VALUE" x="20.32" y="-0.635" size="1.27" layer="27"/>
 </element>
+<element name="SJ4" library="freetronics-jon" package="SJ" value="" x="27.94" y="7.366" rot="MR180"/>
 </elements>
 <signals>
@@
 <wire x1="36.576" y1="25.4" x2="32.512" y2="25.4" width="0.4064" layer="1"/>
 <contactref element="J2" pad="2"/>
-<wire x1="26.162" y1="7.366" x2="28.702" y2="9.906" width="0.4064" layer="16"/>
-<wire x1="28.702" y1="9.906" x2="28.702" y2="21.59" width="0.4064" layer="16"/>
-<wire x1="26.162" y1="7.366" x2="22.606" y2="7.366" width="0.4064" layer="16"/>
+<wire x1="28.702" y1="11.684" x2="28.702" y2="21.59" width="0.4064" layer="16"/>
 <wire x1="17.526" y1="7.366" x2="20.066" y2="7.366" width="0.4064" layer="16"/>
 <wire x1="20.066" y1="7.366" x2="22.606" y2="7.366" width="0.4064" layer="16"/>
-<wire x1="24.13" y1="2.54" x2="24.13" y2="5.842" width="0.4064" layer="16"/>
-<wire x1="24.13" y1="5.842" x2="22.606" y2="7.366" width="0.4064" layer="16"/>
 <wire x1="26.416" y1="7.112" x2="25.4" y2="6.096" width="0.3048" layer="1"/>
 <wire x1="25.4" y1="6.096" x2="25.4" y2="3.81" width="0.3048" layer="1"/>
 <wire x1="25.4" y1="3.81" x2="24.13" y2="2.54" width="0.3048" layer="1"/>
+<contactref element="SJ4" pad="1"/>
+<wire x1="24.13" y1="7.366" x2="22.606" y2="7.366" width="0.4064" layer="16"/>
+<wire x1="28.702" y1="11.684" x2="27.178" y2="10.16" width="0.4064" layer="16"/>
+<wire x1="27.178" y1="10.16" x2="27.178" y2="7.366" width="0.4064" layer="16"/>
+<wire x1="27.178" y1="7.366" x2="25.146" y2="7.366" width="0.4064" layer="16"/>
+<wire x1="25.146" y1="7.366" x2="24.638" y2="6.858" width="0.4064" layer="16"/>
+<wire x1="24.638" y1="6.858" x2="24.13" y2="6.35" width="0.4064" layer="16"/>
+<wire x1="24.13" y1="6.35" x2="24.13" y2="2.54" width="0.4064" layer="16"/>
+<wire x1="24.13" y1="7.366" x2="24.638" y2="6.858" width="0.4064" layer="16"/>
 </signal>
 <signal name="R3_SDA">
@@
 <signal name="5V">
 <contactref element="J2" pad="5"/>
+<contactref element="SJ4" pad="2"/>
+<wire x1="28.702" y1="7.366" x2="30.734" y2="7.366" width="0.4064" layer="16"/>
+<wire x1="30.734" y1="7.366" x2="31.75" y2="6.35" width="0.4064" layer="16"/>
+<wire x1="31.75" y1="6.35" x2="31.75" y2="2.54" width="0.4064" layer="16"/>
 </signal>
 <signal name="N$47">
